File: ReallyTuffKinematic GPS PCB/ReallyTuffKinematic GPS.kicad_sch (KiCad schematic)
At the start: 42 parts, among them J1 Conn_01x05_Pin, J2 Conn_01x06_Pin, SW2 SKRPACE010, SW3 SKRPACE010, U1 ESP32-C3-MINI-1-N4, X1 X322512MSB4SI

Commit message: sync
Parts:
- added BT1: BH-18650-A1AJ006, easyeda2kicad:BAT-TH_BH-18650-A1AJ006, symbol easyeda2kicad:BH-18650-A1AJ006
- added C27: 10nF, Capacitor_SMD:C_0603_1608Metric, symbol Device:C
- added C28, C30: 10uF, Capacitor_SMD:C_0603_1608Metric, symbol Device:C
- added C29, C31, C32: 1uF, Capacitor_SMD:C_0603_1608Metric, symbol Device:C
- added D2, D3: LED, symbol Device:LED
- added D5: USBLC6-2SC6_C2687116, easyeda2kicad:SOT-23-6_L2.9-W1.6-P0.95-LS2.8-BL, symbol easyeda2kicad:USBLC6-2SC6_C2687116
- added R13: 1.2k, Resistor_SMD:R_0603_1608Metric, symbol Device:R
- added R14, R15: 1k, Resistor_SMD:R_0603_1608Metric, symbol Device:R
- added R16: 470, Resistor_SMD:R_0603_1608Metric, symbol Device:R
- added R32, R33: 5.1k, Resistor_SMD:R_0603_1608Metric, symbol Device:R
- added R34, R35: 27, Resistor_SMD:R_0603_1608Metric, symbol Device:R
- added U2: TP4056-42-ESOP8, Package_SO:SOIC-8-1EP_3.9x4.9mm_P1.27mm_EP2.41x3.3mm_ThermalVias, symbol Battery_Management:TP4056-42-ESOP8
- added U3: AP2112K-3.3, Package_TO_SOT_SMD:SOT-23-5, symbol Regulator_Linear:AP2112K-3.3
- added U4: DW03C_C41367942, easyeda2kicad:SOT-23-5_L2.9-W1.6-P0.95-LS2.9-BL, symbol easyeda2kicad:DW03C_C41367942
- added USB1: USB-TYPE-C-018, easyeda2kicad:USB-C_SMD-TYPE-C-31-M-12, symbol easyeda2kicad:USB-TYPE-C-018
Connections:
- net +3.3V: now also R9.2, C32.2, R14.1, R15.1, U3.5 (VOUT); no longer R9.1
- net GND: now also C27.1, C29.2, C30.1, C31.2, C32.1, D5.2 (GND), R13.2, R32.2, R33.1, U2.1 (TEMP), U2.3 (GND), U2.9 (EPAD), U3.2 (GND), U4.4 (VM), USB1.A1 (GND), USB1.A12 (GND), USB1.B1 (GND), USB1.B12 (GND); no longer R11.2, R12.2, U1.22 (IO8), U1.5 (IO2)
- net RP2350_GPIO_1: no longer J2.1 (Pin_1)
- net RP2350_GPIO_2: now also R9.1; no longer R9.2
- net RP2350_GPIO_3: now also J2.4 (Pin_4), U1.23 (IO9)
- net RP2350_USB_DN: now reaches RP2350.51 (USB_DM)
- net RP2350_USB_DN: now also R34.2
- net RP2350_USB_DP: now reaches RP2350.52 (USB_DP)
- net RP2350_USB_DP: now also R35.1
- new net: R12.2, U1.22 (IO8)
- new net: D5.3 (I/O2), R34.1
- new net: R32.1, USB1.A5 (CC1)
- new net: D3.2 (A), R15.2
- new net: D5.4 (I/O2), R35.2
- new net: D2.2 (A), R14.2
- new net: R13.1, U2.2 (PROG)
- new net: D2.1 (K), U2.6 (~{STDBY})
- new net: D3.1 (K), U2.7 (~{CHRG})
- new net: R11.2, U1.5 (IO2)
- new net: C28.2, C29.1
- new net: C27.2, USB1.0 (SH), USB1.1 (SH), USB1.2 (SH), USB1.3 (SH)
- new net: C31.1, R16.2, U4.3 (VDD)
- new net: R33.2, USB1.B5 (CC2)
- new net BATT+: BT1.2, C30.2, R16.1, U2.5 (BAT), U3.1 (VIN), U3.3 (EN)
- new net BATT-: BT1.1, U4.2 (GND)
- new net USB_D+: D5.6 (I/O1), USB1.A6 (DP1), USB1.B6 (DP2)
- new net USB_D-: D5.1 (I/O1), USB1.A7 (DN1), USB1.B7 (DN2)
- new net USB_VBUS: C28.1, D5.5 (VBUS), U2.4 (V_{CC}), U2.8 (CE), USB1.A4 (VBUS), USB1.A9 (VBUS), USB1.B4 (VBUS), USB1.B9 (VBUS)
- no-connect marks 21 -> 23
Other:
- note added: "Batt Connector"
- note added: "Batt Protection"
- note added: "Charger"
- note added: "ESD Protection"
- note added: "ESP32 DEBUG"
- note added: "LDO Regulator"
- note added: "USB-C Connector"
- moved on the sheet: C25, C26, J2, R11, R9

Commit message: sync
Parts:
- added C33: 4.7uF, Capacitor_SMD:C_0603_1608Metric, symbol Device:C
- added C34, C35, C36: 100nF, Capacitor_SMD:C_0603_1608Metric, symbol Device:C
- added IC1: PNT-SG3FS-TR, PNTSG3FSTR, symbol Mouser:PNT-SG3FS-TR
- added R17, R18: 10k, Resistor_SMD:R_0603_1608Metric, symbol Device:R
Connections:
- net +3.3V: now also C34.2, C35.2, C36.2, R17.1
- net GND: now also IC1.1 (GND), IC1.10 (GND_RF_1), IC1.12 (GND_RF_2), R18.2
- net RP2350_GPIO_4: now also IC1.3 (UART-RX)
- net RP2350_GPIO_5: now also IC1.2 (UART-TX)
- net RP2350_GPIO_6: now also IC1.9 (NRESET), R17.2
- net RP2350_GPIO_7: now also IC1.5 (WAKEUP)
- net RP2350_GPIO_8: now also IC1.4 (PPS)
- net RP2350_GPIO_9: now also IC1.13 (ANTOFF), R18.1
- net USB_D+: now also D5.3 (I/O2); no longer D5.6 (I/O1)
- net at R34.1: now also D5.6 (I/O1); no longer D5.3 (I/O2)
- new net: C33.1, IC1.8 (VCC)
- new net: C33.2, C34.1
- new net: C36.1, IC1.6 (VBAT)
- new net: C35.1, IC1.7 (VCC_IO)
- no-connect marks 23 -> 25
Other:
- note added: "GNSS"
- note added: "RX"
- note added: "TX"
- moved on the sheet: D5, R34, R35
