File: PiSat PCB/PiSat.kicad_pcb (KiCad board)
At the start: 4 copper layers, 85 x 56 mm, 87 parts, among them IC1 PNT-SG3FS-TR, J1 Conn_01x05_Pin, J3 Conn_01x06_Pin, Q7 AO3407A, SW1 MSK12C02, SW2 SKRPACE010, SW3 SKRPACE010, U12 AP2112K-3.3, U2 TP4056-42-ESOP8, U4 DW03C_C41367942, U5 SMA-KWE_C7498154, U6 ESP32-C3-MINI-1U-N4, X1 X322512MSB4SI

Commit message: sync
Parts:
- moved R18 3.32 mm to (76.2, 24.0), turned to 90 degrees
- moved C20 1.68 mm to (12.8, 30.8), turned to -90 degrees
- moved C37 1.52 mm to (74.5, 26.2)
- moved R13 1.31 mm to (46.5, 21.2), turned to 180 degrees
- moved C15 1.27 mm to (8.50, 27.8)
- moved L2 0.80 mm to (74.5, 29.2), turned to -90 degrees
- moved C19 0.75 mm to (8.75, 25.5)
Routing:
- net RP2350_GPIO_9: track 2.86 -> 94.7 mm, vias 1 -> 4
- net RP2350_GPIO_2: track 19.1 -> 99.5 mm, vias 1 -> 2
- net RP2350_GPIO_4: track 9.54 -> 89.8 mm
- net RP2350_GPIO_5: track 8.54 -> 87.5 mm
- net RP2350_GPIO_7: track 6.89 -> 81.1 mm
- net RP2350_GPIO_8: track 6.23 -> 78.1 mm
- net RP2350_GPIO_6: track 7.84 -> 76.4 mm, vias 1 -> 2
- net RP2350_GPIO_3: track 13.7 -> 80.5 mm, vias 1 -> 2
- net RP2350_GPIO_0: track 12.7 -> 74.4 mm, vias 1 -> 2
- net RP2350_GPIO_1: track 12.8 -> 74.2 mm, vias 1 -> 2
- net USB_VBUS: track 29.4 -> 69.6 mm
- net GND: track 74.3 -> 94.0 mm, vias 60 -> 89
- net +3.3V: track 51.7 -> 49.8 mm, vias 36 -> 39
- net Net-(U6-IO8): track 0.00 -> 1.74 mm
- net Net-(IC1-VCC_RF): track 3.20 -> 4.70 mm
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
Commit message: sync
Parts:
- moved R3 2.27 mm to (3.00, 9.75), turned to 90 degrees
- moved SW3 1.03 mm to (11.0, 2.50)
- moved U5 0.36 mm to (80.5, 29.7)
- turned C30 to 90 degrees
Connections:
- C30 pad 1: GND -> BATT_SW+
- C30 pad 2: BATT_SW+ -> GND
- D4 pad 1: RP2350_GPIO_10 -> RP2350_GPIO_11
- D6 pad 1: RP2350_GPIO_11 -> RP2350_GPIO_10
Routing:
- net RP2350_GPIO_10: track 2.75 -> 69.0 mm, vias 0 -> 2
- net RP2350_GPIO_11: track 2.82 -> 63.4 mm, vias 0 -> 2
- net RP2350_RUN: track 43.5 -> 73.9 mm, vias 1 -> 2
- net RF_IN: track 0.00 -> 8.85 mm
- net GND: track 94.0 -> 102.6 mm, vias 89 -> 96
- net +1V1: track 29.9 -> 34.9 mm, vias 0 -> 4
- net RP2350_GPIO_8: track 78.1 -> 81.4 mm
- net Net-(R3-Pad2): track 8.13 -> 11.0 mm
- net RP2350_GPIO_9: track 94.7 -> 97.1 mm
- net RP2350_GPIO_7: track 81.1 -> 83.4 mm
- net RP2350_GPIO_5: track 87.5 -> 89.4 mm
- net RP2350_GPIO_4: track 89.8 -> 91.5 mm
- net RP2350_QSPI_SS: track 24.0 -> 22.5 mm
- net RP2350_GPIO_6: track 76.4 -> 77.5 mm
- added copper zone on In2.Cu, net +1V1

Commit message: sync
Parts:
- removed C28, C30: 10uF, Capacitor_SMD:C_0603_1608Metric
- removed C29: 1uF, Capacitor_SMD:C_0603_1608Metric
- removed D2, D3: LED, LED_SMD:LED_0402_1005Metric
- removed R13: 1.2k, Resistor_SMD:R_0603_1608Metric
- removed R14, R15: 1k, Resistor_SMD:R_0603_1608Metric
- removed U2: TP4056-42-ESOP8, Package_SO:SOIC-8-1EP_3.9x4.9mm_P1.27mm_EP2.41x3.3mm_ThermalVias
- added C32: 1uF, Capacitor_SMD:C_0603_1608Metric, F.Cu at (44.5, 26.2)
- added C40: 10uF, Capacitor_SMD:C_0603_1608Metric, F.Cu at (46.5, 30.4)
- added C41: 1uF, Capacitor_SMD:C_0603_1608Metric, F.Cu at (48.0, 30.4)
- added D7: LED, LED_SMD:LED_0402_1005Metric, F.Cu at (53.9, 2.17)
- added D8: LED, LED_SMD:LED_0402_1005Metric, F.Cu at (48.0, 2.08)
- added G***: LOGO, dino:dino, F.Cu at (81.8, 20.0)
- added G***: LOGO, dino:dino, B.Cu at (28.0, 26.0)
- added G***: LOGO, dino:dino, B.Cu at (22.8, 24.0)
- added G***: LOGO, dino:dino, B.Cu at (46.4, 15.6)
- added G***: LOGO, dino:dino, B.Cu at (11.3, 26.7)
- added G***: LOGO, dino:dino, B.Cu at (75.1, 3.80)
- added G***: LOGO, dino:dino, B.Cu at (33.5, 19.0)
- added G***: LOGO, dino:dino, B.Cu at (62.8, 10.7)
- added G***: LOGO, dino:dino, B.Cu at (24.7, 8.81)
- added G***: LOGO, dino:dino, B.Cu at (9.50, 52.8)
- added G***: LOGO, dino:dino, B.Cu at (42.4, 9.95)
- added G***: LOGO, dino:dino, B.Cu at (70.0, 14.0)
- added G***: LOGO, dino:dino, B.Cu at (34.0, 6.46)
- added G***: LOGO, dino:dino, B.Cu at (78.1, 52.8)
- added G***: LOGO, dino:dino, B.Cu at (46.2, 37.6)
- added G***: LOGO, dino:dino, B.Cu at (7.31, 32.1)
- added G***: LOGO, dino:dino, B.Cu at (59.8, 16.5)
- added G***: LOGO, dino:dino, B.Cu at (51.4, 50.3)
- added G***: LOGO, dino:dino, B.Cu at (82.7, 21.4)
- added G***: LOGO, dino:dino, B.Cu at (64.8, 22.8)
- added G***: LOGO, pisat:pisat, B.Cu at (53.9, 58.5)
- added G***: LOGO, dino:dino, B.Cu at (32.9, 40.7)
- added G***: LOGO, dino:dino, B.Cu at (77.5, 10.5)
- added G***: LOGO, dino:dino, B.Cu at (51.5, 4.91)
- added G***: LOGO, dino:dino, B.Cu at (54.4, 19.8)
- added G***: LOGO, dino:dino, B.Cu at (65.0, 30.2)
- added G***: LOGO, dino:dino, B.Cu at (16.2, 36.3)
- added G***: LOGO, dino:dino, B.Cu at (74.5, 22.0)
- added G***: LOGO, dino:dino, B.Cu at (9.45, 13.8)
- added G***: LOGO, dino:dino, B.Cu at (51.5, 26.8)
- added G***: LOGO, dino:dino, B.Cu at (57.1, 18.7)
- added GNU: Symbol_GNU-Logo_SilkscreenTop, Symbol:Symbol_GNU-Logo_SilkscreenTop, B.Cu at (20.5, 46.4)
- added J4: Conn_01x03_Pin, Connector_PinHeader_2.54mm:PinHeader_1x03_P2.54mm_Vertical, F.Cu at (54.5, 13.7)
- added J5: Conn_01x05_Pin, Connector_PinHeader_2.54mm:PinHeader_1x05_P2.54mm_Vertical, F.Cu at (69.5, 12.0)
- added J6: Conn_01x05_Pin, Connector_PinHeader_2.54mm:PinHeader_1x05_P2.54mm_Vertical, F.Cu at (65.9, 1.84)
- added R11: 1.5k, Resistor_SMD:R_0603_1608Metric, F.Cu at (46.1, 27.9)
- added R12: 10k, Resistor_SMD:R_0603_1608Metric, F.Cu at (39.0, 27.9)
- added R24: 1k, Resistor_SMD:R_0603_1608Metric, F.Cu at (56.8, 2.25)
- added R29: 1k, Resistor_SMD:R_0603_1608Metric, F.Cu at (50.8, 2.00)
- added R9: 1k, Resistor_SMD:R_0603_1608Metric, F.Cu at (41.3, 26.2)
- added U1: BQ24075RGTR, easyeda2kicad:QFN-16_L3.0-W3.0-P0.50-TL-EP1.7, F.Cu at (42.2, 29.7)
- added hackclub: LOGO, hackclub:hackclub, B.Cu at (39.0, 47.8)
- moved C65 15.3 mm to (54.8, 21.8), turned to 180 degrees
- moved U12 13.1 mm to (49.9, 21.8), turned to 180 degrees
- moved C38 12.0 mm to (81.2, 2.75), turned to 0 degrees
- moved R20 11.1 mm to (71.0, 15.8), turned to 90 degrees
- moved C39 10.1 mm to (72.3, 3.19), turned to 90 degrees
- moved R19 8.40 mm to (77.9, 3.80), turned to 0 degrees
- moved C1 8.22 mm to (52.2, 25.2), turned to 180 degrees
- moved R10 8.06 mm to (74.7, 3.80), turned to 180 degrees
- moved BUZZER2 5.22 mm to (29.3, 9.50), turned to 180 degrees
- moved C71C1 5.17 mm to (52.2, 27.2), turned to 0 degrees
- moved R27 4.70 mm to (33.5, 8.75), turned to 90 degrees
- moved R35 4.37 mm to (18.5, 14.5)
- moved R34 4.30 mm to (20.0, 14.5)
- moved U6 4.06 mm to (77.8, 11.5), turned to -90 degrees
- moved R25 3.59 mm to (36.0, 27.3), turned to 90 degrees
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- renumbered C71Ceramic1 to C71C1
Connections:
- Q7 pad 2: BATT+ -> BATT_OUT
- R16 pad 1: BATT_SW+ -> BATT+
- R25 pad 1: BATT_SW+ -> BATT+
- R27 pad 1: RP2350_GPIO_22 -> RP2350_GPIO_25
- R28 pad 2: BATT+ -> BATT_OUT
- RP2350 pad 16: unconnected-(RP2350-GPIO12-Pad16) -> RP2350_GPIO_12
- RP2350 pad 17: unconnected-(RP2350-GPIO13-Pad17) -> RP2350_GPIO_13
- RP2350 pad 18: unconnected-(RP2350-GPIO14-Pad18) -> RP2350_GPIO_14
- RP2350 pad 19: unconnected-(RP2350-GPIO15-Pad19) -> RP2350_GPIO_15
- RP2350 pad 31: unconnected-(RP2350-GPIO19-Pad31) -> RP2350_GPIO_19
- RP2350 pad 32: unconnected-(RP2350-GPIO20-Pad32) -> RP2350_GPIO_20
- RP2350 pad 33: unconnected-(RP2350-GPIO21-Pad33) -> RP2350_GPIO_21
- RP2350 pad 35: unconnected-(RP2350-GPIO23-Pad35) -> RP2350_GPIO_23
- RP2350 pad 36: unconnected-(RP2350-GPIO24-Pad36) -> RP2350_GPIO_24
- RP2350 pad 37: unconnected-(RP2350-GPIO25-Pad37) -> RP2350_GPIO_25
- RP2350 pad 41: unconnected-(RP2350-GPIO27/ADC1-Pad41) -> RP2350_GPIO_27_ADC
- RP2350 pad 42: unconnected-(RP2350-GPIO28/ADC2-Pad42) -> RP2350_GPIO_28_ADC
- RP2350 pad 43: unconnected-(RP2350-GPIO29/ADC3-Pad43) -> RP2350_GPIO_29_ADC
Routing:
- net (no net): track 0.00 -> 197.6 mm
- net RP2350_GPIO_13: track 0.00 -> 71.0 mm, vias 0 -> 2
- net RP2350_GPIO_12: track 0.00 -> 69.9 mm, vias 0 -> 2
- net RP2350_GPIO_14: track 0.00 -> 69.6 mm, vias 0 -> 2
- net RP2350_GPIO_24: track 0.00 -> 68.2 mm, vias 0 -> 2
- net RP2350_GPIO_15: track 0.00 -> 68.0 mm, vias 0 -> 2
- net RP2350_GPIO_23: track 0.00 -> 66.6 mm, vias 0 -> 2
- net RP2350_GPIO_21: track 0.00 -> 62.8 mm, vias 0 -> 2
- net RP2350_GPIO_20: track 0.00 -> 60.8 mm, vias 0 -> 2
- net RP2350_GPIO_19: track 0.00 -> 54.4 mm, vias 0 -> 3
- net RP2350_GPIO_29_ADC: track 0.00 -> 48.8 mm, vias 0 -> 3
- net RP2350_GPIO_28_ADC: track 0.00 -> 47.1 mm, vias 0 -> 3
- net RP2350_GPIO_27_ADC: track 0.00 -> 46.8 mm, vias 0 -> 3
- net RP2350_GPIO_22: track 21.4 -> 65.2 mm
- net Net-(D7-K): track 0.00 -> 36.6 mm, vias 0 -> 2
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Other:
- board text added: "12"
- board text added: "13"
- board text added: "14"
- board text added: "15"
- board text added: "19"
- board text added: "20"
- board text added: "21"
- board text added: "22"
- board text added: "23"
- board text added: "24"
- board text added: "27A"
- board text added: "28A"
- board text added: "29A"
- board text added: "CLK"
- board text added: "DIO"
- board text added: "GPIO"
- board text added: "USB"
- board text removed: "STDBY"
