File: PiSat PCB/PiSat.kicad_pcb (KiCad board)
At the start: 4 copper layers, 85 x 56 mm, 125 parts, among them IC1 PNT-SG3FS-TR, J1 Conn_01x05_Pin, J3 Conn_01x06_Pin, J4 Conn_01x03_Pin, J5 Conn_01x05_Pin, J6 Conn_01x05_Pin, Q7 AO3407A, SW1 MSK12C02, SW2 SKRPACE010, SW3 SKRPACE010, U1 BQ24075RGTR, U12 AP2112K-3.3, U4 DW03C_C41367942, U5 SMA-KWE_C7498154, U6 ESP32-C3-MINI-1U-N4, X1 X322512MSB4SI

Commit message: sync
Parts:
- removed D4, D6, D7, D8: LED, LED_SMD:LED_0402_1005Metric
- added LED4: KT-0603R, easyeda2kicad:LED-SMD_L1.6-W0.8-R-RD, F.Cu at (48.0, 2.16)
- added LED5: KT-0603R, easyeda2kicad:LED-SMD_L1.6-W0.8-R-RD, F.Cu at (53.7, 2.16)
- added LED6: KT-0603R, easyeda2kicad:LED-SMD_L1.6-W0.8-R-RD, F.Cu at (54.5, 5.75)
- added LED7: KT-0603R, easyeda2kicad:LED-SMD_L1.6-W0.8-R-RD, F.Cu at (48.6, 5.75)
- moved R21 0.49 mm to (51.5, 5.75)
- moved R22 0.25 mm to (57.4, 5.75)
- moved R29 0.16 mm to (50.7, 2.16)
- moved R24 0.09 mm to (56.7, 2.16)
Routing:
- net +1V1: track 38.5 -> 34.5 mm
- net RP2350_GPIO_11: track 64.8 -> 63.6 mm
