File: PiSat PCB/PiSat.kicad_sch (KiCad schematic)
At the start: 74 parts, among them IC1 PNT-SG3FS-TR, J1 Conn_01x05_Pin, J2 Conn_01x06_Pin, SW2 SKRPACE010, SW3 SKRPACE010, U2 TP4056-42-ESOP8, U3 AP2112K-3.3, U4 DW03C_C41367942, U5 SMA-KWE_C7498154, U6 ESP32-C3-MINI-1U-N4, X1 X322512MSB4SI

Commit message: sync
Parts:
- removed C32: 1uF, Capacitor_SMD:C_0603_1608Metric, symbol Device:C
- removed L2: 47nH, symbol Device:L
- removed U3: AP2112K-3.3, Package_TO_SOT_SMD:SOT-23-5, symbol Regulator_Linear:AP2112K-3.3
- added C1: CL21A226MAQNNNE, easyeda2kicad:C0805, symbol easyeda2kicad:CL21A226MAQNNNE
- added C65: 1uF, Capacitor_SMD:C_0603_1608Metric, symbol Device:C
- added C71: 100nF, Capacitor_SMD:C_0603_1608Metric, symbol Device:C
- added C71Ceramic1: 10uF, Capacitor_SMD:C_0805_2012Metric, symbol Device:C
- added D4, D6: LED, LED_SMD:LED_0402_1005Metric, symbol Device:LED
- added J3: Conn_01x06_Pin, Connector_PinHeader_2.54mm:PinHeader_1x06_P2.54mm_Vertical, symbol Connector:Conn_01x06_Pin
- added L2: LQW15AN47NG00D, easyeda2kicad:L0402, symbol easyeda2kicad:LQW15AN47NG00D
- added Q7: AO3407A, easyeda2kicad:SOT-23-3_L2.9-W1.6-P1.90-LS2.8-BR, symbol easyeda2kicad:AO3407A
- added R21, R22: 1k, Resistor_SMD:R_0603_1608Metric, symbol Device:R
- added R23: 10k, Resistor_SMD:R_0603_1608Metric, symbol Device:R
- added R25, R26: 220k, Resistor_SMD:R_0603_1608Metric, symbol Device:R
- added R28: 100k, Resistor_SMD:R_0603_1608Metric, symbol Device:R
- added SW1: MSK12C02, easyeda2kicad:SW-TH_MSK12C02, symbol easyeda2kicad:MSK12C02
- added U12: AP2112K-3.3, Package_TO_SOT_SMD:SOT-23-5, symbol Regulator_Linear:AP2112K-3.3
- D2, D3: footprint (none) -> LED_SMD:LED_0402_1005Metric
- J1: footprint (none) -> Connector_PinHeader_2.54mm:PinHeader_1x05_P2.54mm_Vertical
Connections:
- net +3.3V: now also R17.2, J3.5 (Pin_5), R21.1, R22.1, U12.5 (VOUT); no longer R17.1
- net BATT+: now also BT1.1, Q7.2 (S), R28.2; no longer BT1.2, C30.2, R16.1, U2.5 (BAT)
- net BATT-: now also BT1.2; no longer BT1.1
- net GND: now also C30.2, C1.2, C65.1, C71.1, C71Ceramic1.1, J3.6 (Pin_6), R26.1, SW1.3, U12.2 (GND); no longer C30.1
- net RF_IN: now also L2.2
- net RP2350_GPIO_0: now also J3.1 (Pin_1)
- net RP2350_GPIO_1: now also J3.2 (Pin_2)
- net RP2350_GPIO_10: now also D4.1 (K)
- net RP2350_GPIO_11: now also D6.1 (K)
- net RP2350_GPIO_2: now also J3.3 (Pin_3)
- net RP2350_GPIO_26_ADC: now also C71.2, R25.2, R26.2
- net RP2350_GPIO_3: now also J3.4 (Pin_4)
- net RP2350_GPIO_6: now also R17.1; no longer R17.2
- net at C37.2, IC1.14 (VCC_RF): now also L2.1
- net RP2350_GPIO_12: no longer names the net of RP2350.16 (GPIO12)
- net RP2350_GPIO_13: no longer names the net of RP2350.17 (GPIO13)
- net RP2350_GPIO_14: no longer names the net of RP2350.18 (GPIO14)
- net RP2350_GPIO_15: no longer names the net of RP2350.19 (GPIO15)
- net RP2350_GPIO_16: no longer names the net of RP2350.27 (GPIO16)
- net RP2350_GPIO_17: no longer names the net of RP2350.28 (GPIO17)
- net RP2350_GPIO_18: no longer names the net of RP2350.29 (GPIO18)
- net RP2350_GPIO_19: no longer names the net of RP2350.31 (GPIO19)
- net RP2350_GPIO_20: no longer names the net of RP2350.32 (GPIO20)
- net RP2350_GPIO_21: no longer names the net of RP2350.33 (GPIO21)
- net RP2350_GPIO_23: no longer names the net of RP2350.35 (GPIO23)
- net RP2350_GPIO_24: no longer names the net of RP2350.36 (GPIO24)
- net RP2350_GPIO_25: no longer names the net of RP2350.37 (GPIO25)
- net RP2350_GPIO_27_ADC: no longer names the net of RP2350.41 (GPIO27/ADC1)
- net RP2350_GPIO_28_ADC: no longer names the net of RP2350.42 (GPIO28/ADC2)
- net RP2350_GPIO_29_ADC: no longer names the net of RP2350.43 (GPIO29/ADC3)
- new net: Q7.1 (G), R23.2, R28.1
- new net: D6.2 (A), R22.2
- new net: D4.2 (A), R21.2
- new net: R23.1, SW1.2
- new net BATT_SW+: C1.1, C30.1, C65.2, C71Ceramic1.2, Q7.3 (D), R16.1, R25.1, U12.1 (VIN), U12.3 (EN), U2.5 (BAT)
- no-connect marks 37 -> 55
Other:
- note added: "3.3V REG"
- note added: "ARM"
- note added: "ESP32-C3 DEBUG"
- note added: "STATUS"
- note added: "V MON"
- note added: "VMON"
- note removed: "LDO Regulator"
- moved on the sheet: C10, C11, C12, C13, C30, C31, R16, R17, U4

Commit message: sync
Connections:
- net BATT+: now also BT1.2; no longer BT1.1
- net BATT-: now also BT1.1; no longer BT1.2
- net RP2350_GPIO_10: now also D6.1 (K); no longer D4.1 (K)
- net RP2350_GPIO_11: now also D4.1 (K); no longer D6.1 (K)
Changed lines of the file:
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@@
+		)
+	)
+	(global_label "RP2350_GPIO_10"
+		(shape input)
+		(at 245.11 195.58 180)
+		(fields_autoplaced yes)
+		(effects
+			(font
+				(size 1.27 1.27)
+			)
+			(justify right)
+		)
+		(property "Intersheetrefs" "${INTERSHEET_REFS}"
+			(at 225.9173 195.58 0)
+			(hide yes)
+			(show_name no)
+			(do_not_autoplace no)
+			(effects
+				(font
+					(size 1.27 1.27)
+				)
+				(justify right)
+			)
 		)
 	)
@@
 	(global_label "RP2350_GPIO_11"
 		(shape input)
-		(at 245.11 195.58 180)
-		(fields_autoplaced yes)
-		(effects
-			(font
-				(size 1.27 1.27)
-			)
-			(justify right)
-		)
-		(property "Intersheetrefs" "${INTERSHEET_REFS}"
-			(at 225.9173 195.58 0)
+		(at 251.46 184.15 180)
+		(fields_autoplaced yes)
+		(effects
+			(font
+				(size 1.27 1.27)
+			)
+			(justify right)
+		)
+		(property "Intersheetrefs" "${INTERSHEET_REFS}"
+			(at 232.2673 184.15 0)
 			(hide yes)
 			(show_name no)
@@
 		(property "Intersheetrefs" "${INTERSHEET_REFS}"
 			(at 31.9701 255.27 0)
-			(hide yes)
-			(show_name no)
-			(do_not_autoplace no)
-			(effects
-				(font
-					(size 1.27 1.27)
-				)
-				(justify right)
-			)
-		)
-	)
-	(global_label "RP2350_GPIO_10"
-		(shape input)
-		(at 251.46 184.15 180)
-		(fields_autoplaced yes)
-		(effects
-			(font
-				(size 1.27 1.27)
-			)
-			(justify right)
-		)
-		(property "Intersheetrefs" "${INTERSHEET_REFS}"
-			(at 232.2673 184.15 0)
 			(hide yes)
 			(show_name no)
@@
 		(lib_id "easyeda2kicad:BH-18650-A1AJ006")
 		(at 184.15 163.83 0)
-		(mirror y)
+		(mirror x)
 		(unit 1)
 		(body_style 1)
@@
 		(dnp no)
 		(property "Reference" "BT1"
+			(at 184.15 159.766 0)
+			(show_name no)
+			(do_not_autoplace no)
+			(effects
+				(font
+					(size 1.27 1.27)
+				)
+			)
+		)
+		(property "Value" "BH-18650-A1AJ006"
+			(at 184.15 157.226 0)
+			(show_name no)
+			(do_not_autoplace no)
+			(effects
+				(font
+					(size 1.27 1.27)
+				)
+			)
+		)
+		(property "Footprint" "easyeda2kicad:BAT-TH_BH-18650-A1AJ006"
 			(at 184.15 156.21 0)
-			(show_name no)
-			(do_not_autoplace no)
-			(effects
-				(font
-					(size 1.27 1.27)
-				)
-			)
-		)
-		(property "Value" "BH-18650-A1AJ006"
-			(at 184.15 158.75 0)
-			(show_name no)
-			(do_not_autoplace no)
-			(effects
-				(font
-					(size 1.27 1.27)
-				)
-			)
-		)
-		(property "Footprint" "easyeda2kicad:BAT-TH_BH-18650-A1AJ006"
-			(at 184.15 171.45 0)
 			(hide yes)
 			(show_name no)
@@
 		)
 		(property "Datasheet" "https://www.lcsc.com/datasheet/C5290175.pdf"
-			(at 184.15 173.99 0)
+			(at 184.15 153.67 0)
 			(hide yes)
 			(show_name no)
@@
 		)
 		(property "Manufacturer" "MYOUNG(美阳)"
-			(at 184.15 176.53 0)
+			(at 184.15 151.13 0)
 			(hide yes)
 			(show_name no)
@@
 		)
 		(property "MPN" "BH-18650-A1AJ006"
-			(at 184.15 179.07 0)
+			(at 184.15 148.59 0)
 			(hide yes)
 			(show_name no)
@@
 		)
 		(property "LCSC Part" "C5290175"
-			(at 184.15 181.61 0)
-			(hide yes)
-			(show_name no)
+			(at 184.15 146.05 0)
+			(hide yes)
+			(show_name no)

Commit message: sync
Parts:
- removed C28, C30: 10uF, Capacitor_SMD:C_0603_1608Metric, symbol Device:C
- removed C29: 1uF, Capacitor_SMD:C_0603_1608Metric, symbol Device:C
- removed D2, D3: LED, LED_SMD:LED_0402_1005Metric, symbol Device:LED
- removed J2: Conn_01x06_Pin, symbol Connector:Conn_01x06_Pin
- removed R13: 1.2k, Resistor_SMD:R_0603_1608Metric, symbol Device:R
- removed R14, R15: 1k, Resistor_SMD:R_0603_1608Metric, symbol Device:R
- removed U2: TP4056-42-ESOP8, Package_SO:SOIC-8-1EP_3.9x4.9mm_P1.27mm_EP2.41x3.3mm_ThermalVias, symbol Battery_Management:TP4056-42-ESOP8
- added C32, C41: 1uF, Capacitor_SMD:C_0603_1608Metric, symbol Device:C
- added C40: 10uF, Capacitor_SMD:C_0603_1608Metric, symbol Device:C
- added D7, D8: LED, LED_SMD:LED_0402_1005Metric, symbol Device:LED
- added J4: Conn_01x03_Pin, Connector_PinHeader_2.54mm:PinHeader_1x03_P2.54mm_Vertical, symbol Connector:Conn_01x03_Pin
- added J5, J6: Conn_01x05_Pin, Connector_PinHeader_2.54mm:PinHeader_1x05_P2.54mm_Vertical, symbol Connector:Conn_01x05_Pin
- added R11: 1.5k, Resistor_SMD:R_0603_1608Metric, symbol Device:R
- added R12: 10k, Resistor_SMD:R_0603_1608Metric, symbol Device:R
- added R24, R29, R9: 1k, Resistor_SMD:R_0603_1608Metric, symbol Device:R
- added U1: BQ24075RGTR, easyeda2kicad:QFN-16_L3.0-W3.0-P0.50-TL-EP1.7, symbol easyeda2kicad:BQ24075RGTR
- renumbered C71Ceramic1 to C71C1
Connections:
- net +3.3V: now also R24.1, R29.1
- net BATT+: now also R16.1, R25.1, U1.2 (BAT), U1.3 (BAT); no longer Q7.2 (S), R28.2
- net BATT_SW+: no longer R16.1, R25.1
- net GND: now also C32.1, C41.1, R11.2, R12.2, R9.2, U1.15 (SYSOFF), U1.17 (EP), U1.4 (#CE), U1.6 (EN1), U1.8 (VSS)
- net RP2350_GPIO_22: now also J5.3 (Pin_3); no longer R27.1
- net USB_VBUS: now also C32.2, U1.13 (IN)
- net RP2350_GPIO_12: now reaches RP2350.16 (GPIO12)
- net RP2350_GPIO_12: now also J6.1 (Pin_1)
- net RP2350_GPIO_13: now reaches RP2350.17 (GPIO13)
- net RP2350_GPIO_13: now also J6.2 (Pin_2)
- net RP2350_GPIO_14: now reaches RP2350.18 (GPIO14)
- net RP2350_GPIO_14: now also J6.3 (Pin_3)
- net RP2350_GPIO_15: now reaches RP2350.19 (GPIO15)
- net RP2350_GPIO_15: now also J6.4 (Pin_4)
- net RP2350_GPIO_19: now reaches RP2350.31 (GPIO19)
- net RP2350_GPIO_19: now also J6.5 (Pin_5)
- net RP2350_GPIO_20: now reaches RP2350.32 (GPIO20)
- net RP2350_GPIO_20: now also J5.1 (Pin_1)
- net RP2350_GPIO_21: now reaches RP2350.33 (GPIO21)
- net RP2350_GPIO_21: now also J5.2 (Pin_2)
- net RP2350_GPIO_23: now reaches RP2350.35 (GPIO23)
- net RP2350_GPIO_23: now also J5.4 (Pin_4)
- net RP2350_GPIO_24: now reaches RP2350.36 (GPIO24)
- net RP2350_GPIO_24: now also J5.5 (Pin_5)
- net RP2350_GPIO_25: now reaches RP2350.37 (GPIO25)
- net RP2350_GPIO_25: now also R27.1
- net RP2350_GPIO_27_ADC: now reaches RP2350.41 (GPIO27/ADC1)
- net RP2350_GPIO_27_ADC: now also J4.1 (Pin_1)
- net RP2350_GPIO_28_ADC: now reaches RP2350.42 (GPIO28/ADC2)
- net RP2350_GPIO_28_ADC: now also J4.2 (Pin_2)
- net RP2350_GPIO_29_ADC: now reaches RP2350.43 (GPIO29/ADC3)
- net RP2350_GPIO_29_ADC: now also J4.3 (Pin_3)
- new net: R9.1, U1.16 (ISET)
- new net: D8.1 (K), U1.7 (#PGOOD)
- new net: D8.2 (A), R29.2
- new net: R11.1, U1.12 (ILIM)
- new net: D7.1 (K), U1.9 (#CHG)
- new net: D7.2 (A), R24.2
- new net: R12.1, U1.1 (TS)
- new net: C40.2, C41.2
- new net BATT_OUT: C40.1, Q7.2 (S), R28.2, U1.10 (OUT), U1.11 (OUT), U1.5 (EN2)
- no-connect marks 55 -> 43
Other:
- note added: "GPIO BREAKOUT"
- note added: "difficult to wire"
- note removed: "ESP32 DEBUG"
- moved on the sheet: D4, D6, J3, R21, R22
