File: PiSat PCB/PiSat.kicad_sch (KiCad schematic)
At the start: 92 parts, among them IC1 PNT-SG3FS-TR, J1 Conn_01x05_Pin, J3 Conn_01x06_Pin, J4 Conn_01x03_Pin, J5 Conn_01x05_Pin, J6 Conn_01x05_Pin, Q7 AO3407A, SW1 MSK12C02, SW2 SKRPACE010, SW3 SKRPACE010, U1 BQ24075RGTR, U12 AP2112K-3.3, U4 DW03C_C41367942, U5 SMA-KWE_C7498154, U6 ESP32-C3-MINI-1U-N4, X1 X322512MSB4SI

Commit message: sync
Parts:
- removed D4, D6, D7, D8: LED, LED_SMD:LED_0402_1005Metric, symbol Device:LED
- added LED4, LED5, LED6, LED7: KT-0603R, easyeda2kicad:LED-SMD_L1.6-W0.8-R-RD, symbol easyeda2kicad:KT-0603R
Connections:
- net RP2350_GPIO_10: now also LED6.2 (K)
- net RP2350_GPIO_11: now also LED7.2 (K)
- net at U1.7 (#PGOOD): now also LED4.2 (K)
- net at R29.2: now also LED4.1 (A)
- net at R22.2: now also LED6.1 (A)
- net at U1.9 (#CHG): now also LED5.2 (K)
- net at R24.2: now also LED5.1 (A)
- net at R21.2: now also LED7.1 (A)
Other:
- moved on the sheet: R21, R22, R24, R29

Commit message: sync
Connections:
- net GND: now also U1.14 (TMR)
- no-connect marks 43 -> 42
Changed lines of the file:
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@@
 	)
 	(no_connect
-		(at 152.4 166.37)
-	)
-	(no_connect
 		(at 261.62 54.61)
 	)
@@
 					(unit 1)
 				)
+			)
+		)
+	)
+	(symbol
+		(lib_id "power:GND")
+		(at 152.4 166.37 0)
+		(unit 1)
+		(body_style 1)
+		(exclude_from_sim no)
+		(in_bom yes)
+		(on_board yes)
+		(in_pos_files yes)
+		(dnp no)
+		(property "Reference" "#PWR093"
+			(at 152.4 172.72 0)
+			(hide yes)
+			(show_name no)
+			(do_not_autoplace no)
+			(effects
+				(font
+					(size 1.27 1.27)
+				)
+			)
+		)
+		(property "Value" "GND"
+			(at 149.606 169.418 0)
+			(show_name no)
+			(do_not_autoplace no)
+			(effects
+				(font
+					(size 1.27 1.27)
+				)
+			)
+		)
+		(property "Footprint" ""
+			(at 152.4 166.37 0)
+			(hide yes)
+			(show_name no)
+			(do_not_autoplace no)
+			(effects
+				(font
+					(size 1.27 1.27)
+				)
+			)
+		)
+		(property "Datasheet" ""
+			(at 152.4 166.37 0)
+			(hide yes)
+			(show_name no)
+			(do_not_autoplace no)
+			(effects
+				(font
+					(size 1.27 1.27)
+				)
+			)
+		)
+		(property "Description" "Power symbol creates a global label with name \"GND\" , ground"
+			(at 152.4 166.37 0)
+			(hide yes)
+			(show_name no)
+			(do_not_autoplace no)
+			(effects
+				(font
+					(size 1.27 1.27)
+				)
+			)
+		)
+		(pin "1"
+		)
+		(instances
+			(project "PiSat"
+				(path "/63755c59-753c-4530-b223-ae03b8994baf"
+					(reference "#PWR093")
+					(unit 1)
+				)
